Commit message: Moveit2 Added

File: panda_description/urdf/arm.xacro (robot description, xacro)
@@ -1,4 +1,7 @@
 <?xml version="1.0" ?>
 <robot name="panda" xmlns:xacro="http://www.ros.org/wiki/xacro">
+  <material name="cream">
+    <color rgba="1.000 0.980 0.850 1.000"/>
+  </material>
   <!-- Link 0 - Base -->
   <link name="panda_link0">
@@ -52,5 +55,5 @@
     <child link="panda_link1"/>
     <axis xyz="0 0 1"/>
-    <limit effort="87" lower="-2.9671" upper="2.9671" velocity="2.1750"/>
+    <limit effort="30.0" lower="-2.9671" upper="2.9671" velocity="10.0"/>
   </joint>
   <!-- Link 2 -->
@@ -83,5 +86,5 @@
     <child link="panda_link2"/>
     <axis xyz="0 0 1"/>
-    <limit effort="87" lower="-1.8326" upper="1.8326" velocity="2.1750"/>
+    <limit effort="30.0" lower="-1.8326" upper="1.8326" velocity="10.0"/>
   </joint>
   <!-- Link 3 -->
@@ -114,5 +117,5 @@
     <child link="panda_link3"/>
     <axis xyz="0 0 1"/>
-    <limit effort="87" lower="-2.9671" upper="2.9671" velocity="2.1750"/>
+    <limit effort="30.0" lower="-2.9671" upper="2.9671" velocity="10.0"/>
   </joint>
   <!-- Link 4 -->
@@ -145,5 +148,5 @@
     <child link="panda_link4"/>
     <axis xyz="0 0 1"/>
-    <limit effort="87" lower="-3.1416" upper="0.0" velocity="2.1750"/>
+    <limit effort="30.0" lower="-3.1416" upper="0.0" velocity="10.0"/>
   </joint>
   <!-- Link 5 -->
@@ -176,5 +179,5 @@
     <child link="panda_link5"/>
     <axis xyz="0 0 1"/>
-    <limit effort="12" lower="-2.9671" upper="2.9671" velocity="2.6100"/>
+    <limit effort="30.0" lower="-2.9671" upper="2.9671" velocity="10.0"/>
   </joint>
   <!-- Link 6 -->
@@ -207,5 +210,5 @@
     <child link="panda_link6"/>
     <axis xyz="0 0 1"/>
-    <limit effort="12" lower="-0.0873" upper="3.8223" velocity="2.6100"/>
+    <limit effort="30.0" lower="-0.0873" upper="3.8223" velocity="10.0"/>
   </joint>
   <!-- Link 7 -->
@@ -238,5 +241,5 @@
     <child link="panda_link7"/>
     <axis xyz="0 0 1"/>
-    <limit effort="12" lower="-2.9671" upper="2.9671" velocity="2.6100"/>
+    <limit effort="30.0" lower="-2.9671" upper="2.9671" velocity="10.0"/>
   </joint>
   <!-- Link 8 - No visual/collision, but needs inertial for Gazebo -->
@@ -337,5 +340,5 @@
     <origin rpy="0 0 0" xyz="0 0 0.0584"/>
     <axis xyz="0 1 0"/>
-    <limit effort="20" lower="0.0" upper="0.04" velocity="0.2"/>
+    <limit effort="30.0" lower="0.0" upper="0.04" velocity="10.0"/>
   </joint>
   <!-- Finger Joint 2 -->
@@ -344,7 +347,7 @@
     <child link="panda_rightfinger"/>
     <origin rpy="0 0 0" xyz="0 0 0.0584"/>
-    <axis xyz="0 -1 0"/>
-    <limit effort="20" lower="0.0" upper="0.04" velocity="0.2"/>
-    <mimic joint="panda_finger_joint1"/>
+    <axis xyz="0 1 0"/>
+    <limit effort="30.0" lower="0.0" upper="0.04" velocity="10.0"/>
+    <mimic joint="panda_finger_joint1" multiplier="-1"/>
   </joint>
   <link name="world"/>

File: panda_description/urdf/panda.urdf.xacro (robot description, xacro)
@@ -1,5 +1,4 @@
 <?xml version="1.0"?>
 <robot name="panda" xmlns:xacro="http://www.ros.org/wiki/xacro">
-  <xacro:include filename="$(find panda_description)/urdf/materials.xacro" />
   <xacro:include filename="$(find panda_description)/urdf/arm.xacro" />
   <xacro:include filename="$(find panda_description)/urdf/sensors.xacro" />

Commit message: update

File: panda_description/urdf/arm.xacro (robot description, xacro)
@@ -1,50 +1,50 @@
 <?xml version="1.0" ?>
 <robot name="panda" xmlns:xacro="http://www.ros.org/wiki/xacro">
-  <material name="cream">
-    <color rgba="1.000 0.980 0.850 1.000"/>
+  <material name="red">
+    <color rgba="1.0 0.0 0.0 1.000"/>
   </material>
+  <!-- World Frame -->
+  <link name="world"/>
   <!-- Link 0 - Base -->
   <link name="panda_link0">
     <visual>
       <geometry>
+        <mesh filename="package://panda_description/meshes/visual/link0.dae"/>
+      </geometry>
+    </visual>
+    <collision>
+      <geometry>
         <mesh filename="package://panda_description/meshes/collision/link0.obj"/>
       </geometry>
-      <material name="cream"/>
-    </visual>
-    <collision>
-      <geometry>
-        <mesh filename="package://panda_description/meshes/collision/link0.obj"/>
-      </geometry>
-      <material name="cream"/>
-    </collision>
-    <inertial>
-      <origin xyz="0.0 0.0 0.05" rpy="0 0 0"/>
-      <mass value="2.95"/>
-      <inertia ixx="0.00315" ixy="0.0" ixz="0.0"
-               iyy="0.00315" iyz="0.0"
-               izz="0.004875"/>
-    </inertial>
-  </link>
+    </collision>
+      <inertial>
+          <origin xyz="0 0 0" rpy="0.0 0.0 0.0"/>
+          <mass value="0.1"/>
+          <inertia ixx="0.1" ixy="0.0" ixz="0.0" iyy="0.1" iyz="0.0" izz="0.1"/>
+      </inertial>
+  </link>
+  <!-- World-Base Joint -->
+  <joint name="virtual_joint" type="fixed">
+    <parent link="world"/>
+    <child link="panda_link0"/>
+    <origin xyz="0.6 0 0.35" rpy="0 0 1.57"/>
+  </joint>
   <!-- Link 1 -->
   <link name="panda_link1">
     <visual>
       <geometry>
+        <mesh filename="package://panda_description/meshes/visual/link1.dae"/>
+      </geometry>
+    </visual>
+    <collision>
+      <geometry>
         <mesh filename="package://panda_description/meshes/collision/link1.obj"/>
       </geometry>
-      <material name="cream"/>
-    </visual>
-    <collision>
-      <geometry>
-        <mesh filename="package://panda_description/meshes/collision/link1.obj"/>
-      </geometry>
-      <material name="cream"/>
-    </collision>
-    <inertial>
-      <origin xyz="0.0 -0.032 -0.067" rpy="0 0 0"/>
-      <mass value="2.74"/>
-      <inertia ixx="0.0180" ixy="0.0" ixz="0.0"
-               iyy="0.0193" iyz="0.0014"
-               izz="0.0068"/>
-    </inertial>
+    </collision>
+        <inertial>
+            <origin xyz="0 0 0" rpy="0.0 0.0 0.0"/>
+            <mass value="0.1"/>
+            <inertia ixx="0.1" ixy="0.0" ixz="0.0" iyy="0.1" iyz="0.0" izz="0.1"/>
+        </inertial>
   </link>
   <!-- Joint 1 -->
@@ -61,21 +61,17 @@
     <visual>
       <geometry>
+        <mesh filename="package://panda_description/meshes/visual/link2.dae"/>
+      </geometry>
+    </visual>
+    <collision>
+      <geometry>
         <mesh filename="package://panda_description/meshes/collision/link2.obj"/>
       </geometry>
-      <material name="cream"/>
-    </visual>
-    <collision>
-      <geometry>
-        <mesh filename="package://panda_description/meshes/collision/link2.obj"/>
-      </geometry>
-      <material name="cream"/>
-    </collision>
-    <inertial>
-      <origin xyz="0.0 0.0 0.0" rpy="0 0 0"/>
-      <mass value="2.74"/>
-      <inertia ixx="0.0180" ixy="0.0" ixz="0.0"
-               iyy="0.0068" iyz="0.0"
-               izz="0.0193"/>
-    </inertial>
+    </collision>
+        <inertial>
+          <origin xyz="0 0 0" rpy="0.0 0.0 0.0"/>
+          <mass value="0.1"/>
+          <inertia ixx="0.1" ixy="0.0" ixz="0.0" iyy="0.1" iyz="0.0" izz="0.1"/>
+      </inertial>
   </link>
   <!-- Joint 2 -->
@@ -92,21 +88,17 @@
     <visual>
       <geometry>
+        <mesh filename="package://panda_description/meshes/visual/link3.dae"/>
+      </geometry>
+    </visual>
+    <collision>
+      <geometry>
         <mesh filename="package://panda_description/meshes/collision/link3.obj"/>
       </geometry>
-      <material name="cream"/>
-    </visual>
-    <collision>
-      <geometry>
-        <mesh filename="package://panda_description/meshes/collision/link3.obj"/>
-      </geometry>
-      <material name="cream"/>
-    </collision>
-    <inertial>
-      <origin xyz="0.0434 0.0 -0.121" rpy="0 0 0"/>
-      <mass value="2.38"/>
-      <inertia ixx="0.0125" ixy="0.0" ixz="-0.0036"
-               iyy="0.0165" iyz="0.0"
-               izz="0.0060"/>
-    </inertial>
+    </collision>
+      <inertial>
+          <origin xyz="0 0 0" rpy="0.0 0.0 0.0"/>
+          <mass value="0.1"/>
+          <inertia ixx="0.1" ixy="0.0" ixz="0.0" iyy="0.1" iyz="0.0" izz="0.1"/>
+      </inertial>
   </link>
   <!-- Joint 3 -->
@@ -123,21 +115,17 @@
     <visual>
       <geometry>
+        <mesh filename="package://panda_description/meshes/visual/link4.dae"/>
+      </geometry>
+    </visual>
+    <collision>
+      <geometry>
         <mesh filename="package://panda_description/meshes/collision/link4.obj"/>
       </geometry>
-      <material name="cream"/>
-    </visual>
-    <collision>
-      <geometry>
-        <mesh filename="package://panda_description/meshes/collision/link4.obj"/>
-      </geometry>
-      <material name="cream"/>
-    </collision>
-    <inertial>
-      <origin xyz="0.0 0.0610 -0.104" rpy="0 0 0"/>
-      <mass value="2.74"/>
-      <inertia ixx="0.0358" ixy="0.0" ixz="0.0"
-               iyy="0.0095" iyz="0.0119"
-               izz="0.0304"/>
-    </inertial>
+    </collision>
+      <inertial>
+          <origin xyz="0 0 0" rpy="0.0 0.0 0.0"/>
+          <mass value="0.1"/>
+          <inertia ixx="0.1" ixy="0.0" ixz="0.0" iyy="0.1" iyz="0.0" izz="0.1"/>
+      </inertial>
   </link>
   <!-- Joint 4 -->
@@ -154,21 +142,17 @@
     <visual>
       <geometry>
+        <mesh filename="package://panda_description/meshes/visual/link5.dae"/>
+      </geometry>
+    </visual>
+    <collision>
+      <geometry>
         <mesh filename="package://panda_description/meshes/collision/link5.obj"/>
       </geometry>
-      <material name="cream"/>
-    </visual>
-    <collision>
-      <geometry>
-        <mesh filename="package://panda_description/meshes/collision/link5.obj"/>
-      </geometry>
-      <material name="cream"/>
-    </collision>
-    <inertial>
-      <origin xyz="0.0 0.0610 -0.104" rpy="0 0 0"/>
-      <mass value="2.74"/>
-      <inertia ixx="0.0358" ixy="0.0" ixz="0.0"
-               iyy="0.0095" iyz="0.0119"
-               izz="0.0304"/>
-    </inertial>
+    </collision>
+      <inertial>
+          <origin xyz="0 0 0" rpy="0.0 0.0 0.0"/>
+          <mass value="0.1"/>
+          <inertia ixx="0.1" ixy="0.0" ixz="0.0" iyy="0.1" iyz="0.0" izz="0.1"/>
+      </inertial>
   </link>
   <!-- Joint 5 -->
@@ -185,21 +169,17 @@
     <visual>
       <geometry>
+        <mesh filename="package://panda_description/meshes/visual/link6.dae"/>
+      </geometry>
+    </visual>
+    <collision>
+      <geometry>
         <mesh filename="package://panda_description/meshes/collision/link6.obj"/>
       </geometry>
-      <material name="cream"/>
-    </visual>
-    <collision>
-      <geometry>
-        <mesh filename="package://panda_description/meshes/collision/link6.obj"/>
-      </geometry>
-      <material name="cream"/>
-    </collision>
-    <inertial>
-      <origin xyz="0.051 0.009 -0.015" rpy="0 0 0"/>
-      <mass value="1.55"/>
-      <inertia ixx="0.0047" ixy="0.0" ixz="0.0015"
-               iyy="0.0047" iyz="0.0"
-               izz="0.0031"/>
-    </inertial>
+    </collision>
+      <inertial>
+          <origin xyz="0 0 0" rpy="0.0 0.0 0.0"/>
+          <mass value="0.1"/>
+          <inertia ixx="0.1" ixy="0.0" ixz="0.0" iyy="0.1" iyz="0.0" izz="0.1"/>
+      </inertial>
   </link>
   <!-- Joint 6 -->
@@ -216,21 +196,17 @@
     <visual>
       <geometry>
+        <mesh filename="package://panda_description/meshes/visual/link7.dae"/>
+      </geometry>
+    </visual>
+    <collision>
+      <geometry>
         <mesh filename="package://panda_description/meshes/collision/link7.obj"/>
       </geometry>
-      <material name="cream"/>
-    </visual>
-    <collision>
-      <geometry>
-        <mesh filename="package://panda_description/meshes/collision/link7.obj"/>
-      </geometry>
-      <material name="cream"/>
-    </collision>
-    <inertial>
-      <origin xyz="0.0 0.0 0.02" rpy="0 0 0"/>
-      <mass value="0.54"/>
-      <inertia ixx="0.0012" ixy="0.0" ixz="0.0"
-               iyy="0.0012" iyz="0.0"
-               izz="0.0016"/>
-    </inertial>
+    </collision>
+      <inertial>
+          <origin xyz="0 0 0" rpy="0.0 0.0 0.0"/>
+          <mass value="0.1"/>
+          <inertia ixx="0.1" ixy="0.0" ixz="0.0" iyy="0.1" iyz="0.0" izz="0.1"/>
+      </inertial>
   </link>
   <!-- Joint 7 -->
@@ -243,70 +219,45 @@
     <limit effort="30.0" lower="-2.9671" upper="2.9671" velocity="10.0"/>
   </joint>
-  <!-- Link 8 - No visual/collision, but needs inertial for Gazebo -->
-  <link name="panda_link8">
-    <inertial>
-      <origin xyz="0.0 0.0 0.0" rpy="0 0 0"/>
-      <mass value="0.001"/>
-      <inertia ixx="0.0001" ixy="0.0" ixz="0.0"
-               iyy="0.0001" iyz="0.0"
-               izz="0.0001"/>
-    </inertial>
-  </link>
-  <!-- Joint 8 -->
-  <joint name="panda_joint8" type="fixed">
-    <origin rpy="0 0 0" xyz="0 0 0.107"/>
-    <parent link="panda_link7"/>
-    <child link="panda_link8"/>
-    <axis xyz="0 0 0"/>
-  </joint>
+  <!-- Hand Link -->
+  <link name="panda_hand">
+    <visual>
+      <geometry>
+        <mesh filename="package://panda_description/meshes/visual/hand.dae"/>
+      </geometry>
+    </visual>
+    <collision>
+      <geometry>
+        <mesh filename="package://panda_description/meshes/collision/hand.obj"/>
+      </geometry>
+    </collision>
+      <inertial>
+          <origin xyz="0 0 0" rpy="0.0 0.0 0.0"/>
+          <mass value="0.1"/>
+          <inertia ixx="0.1" ixy="0.0" ixz="0.0" iyy="0.1" iyz="0.0" izz="0.1"/>
+      </inertial>
+  </link>
   <!-- Hand Joint -->
   <joint name="panda_hand_joint" type="fixed">
-    <parent link="panda_link8"/>
+    <parent link="panda_link7"/>
     <child link="panda_hand"/>
-    <origin rpy="0 0 -0.785398163397" xyz="0 0 0"/>
-  </joint>
-  <!-- Hand Link -->
-  <link name="panda_hand">
-    <visual>
-      <geometry>
-        <mesh filename="package://panda_description/meshes/collision/hand.obj"/>
-      </geometry>
-      <material name="cream"/>
-    </visual>
-    <collision>
-      <geometry>
-        <mesh filename="package://panda_description/meshes/collision/hand.obj"/>
-      </geometry>
-      <material name="cream"/>
-    </collision>
-    <inertial>
-      <origin xyz="0.0 0.0 0.05" rpy="0 0 0"/>
-      <mass value="0.76"/>
-      <inertia ixx="0.001" ixy="0.0" ixz="0.0"
-               iyy="0.0025" iyz="0.0"
-               izz="0.0017"/>
-    </inertial>
-  </link>
+    <origin rpy="0 0 -0.785398163397" xyz="0 0 0.106"/>
+  </joint>
   <!-- Left Finger Link -->
   <link name="panda_leftfinger">
     <visual>
       <geometry>
+        <mesh filename="package://panda_description/meshes/visual/finger.dae"/>
+      </geometry>
+    </visual>
+    <collision>
+      <geometry>
         <mesh filename="package://panda_description/meshes/collision/finger.obj"/>
       </geometry>
-      <material name="cream"/>
-    </visual>
-    <collision>
-      <geometry>
-        <mesh filename="package://panda_description/meshes/collision/finger.obj"/>
-      </geometry>
-      <material name="cream"/>
-    </collision>
-    <inertial>
-      <origin xyz="0.0 0.0145 0.0227" rpy="0 0 0"/>
-      <mass value="0.015"/>
-      <inertia ixx="0.0001" ixy="0.0" ixz="0.0"
-               iyy="0.0001" iyz="0.0"
-               izz="0.0001"/>
-    </inertial>
+    </collision>
+      <inertial>
+          <origin xyz="0 0 0" rpy="0.0 0.0 0.0"/>
+          <mass value="0.1"/>
+          <inertia ixx="0.1" ixy="0.0" ixz="0.0" iyy="0.1" iyz="0.0" izz="0.1"/>
+      </inertial>
   </link>
   <!-- Right Finger Link -->
@@ -315,22 +266,18 @@
       <origin rpy="0 0 3.14159265359" xyz="0 0 0"/>
       <geometry>
+        <mesh filename="package://panda_description/meshes/visual/finger.dae"/>
+      </geometry>
+    </visual>
+    <collision>
+      <origin rpy="0 0 3.14159265359" xyz="0 0 0"/>
+      <geometry>
         <mesh filename="package://panda_description/meshes/collision/finger.obj"/>
       </geometry>
-      <material name="cream"/>
-    </visual>
-    <collision>
-      <origin rpy="0 0 3.14159265359" xyz="0 0 0"/>
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
File: panda_description/urdf/gazebo.xacro (robot description, xacro)
@@ -22,26 +22,3 @@
     </xacro:unless>
   </gazebo>
-    <gazebo reference="camera_link">
-        <sensor name="camera" type="camera">
-            <pose>0 0 0 0 1.57 0</pose>
-            <visualize>true</visualize>
-            <update_rate>10.0</update_rate>
-            <alwaysOn>true</alwaysOn>
-            <topic>camera/image_raw</topic>
-            <gz_frame_id>camera_link_optical</gz_frame_id>
-            <camera name="intel_realsense_r200">
-                <camera_info_topic>camera/camera_info</camera_info_topic>
-                <horizontal_fov>1.3962634</horizontal_fov>
-                <image>
-                    <width>640</width>
-                    <height>480</height>
-                    <format>R8G8B8</format>
-                </image>
-                <clip>
-                    <near>0.05</near>
-                    <far>8.0</far>
-                </clip>
-            </camera>
-        </sensor>
-  </gazebo>
 </robot>

File: panda_description/urdf/panda.urdf.xacro (robot description, xacro)
@@ -2,5 +2,5 @@
 <robot name="panda" xmlns:xacro="http://www.ros.org/wiki/xacro">
   <xacro:include filename="$(find panda_description)/urdf/arm.xacro" />
-  <xacro:include filename="$(find panda_description)/urdf/sensors.xacro" />
+  <!-- <xacro:include filename="$(find panda_description)/urdf/sensors.xacro" /> -->
   <xacro:include filename="$(find panda_description)/urdf/gazebo.xacro" />
   <xacro:include filename="$(find panda_description)/urdf/ros2control.xacro" />

File: panda_description/urdf/ros2control.xacro (robot description, xacro)
@@ -23,5 +23,4 @@
       </command_interface>
       <state_interface name="position"/>
-      <state_interface name="velocity"/>
     </joint>
     <!-- Joint 2 -->
@@ -32,5 +31,4 @@
       </command_interface>
       <state_interface name="position"/>
-      <state_interface name="velocity"/>
     </joint>
     <!-- Joint 3 -->
@@ -41,5 +39,4 @@
       </command_interface>
       <state_interface name="position"/>
-      <state_interface name="velocity"/>
     </joint>
     <!-- Joint 4 -->
@@ -50,5 +47,4 @@
       </command_interface>
       <state_interface name="position"/>
-      <state_interface name="velocity"/>
     </joint>
     <!-- Joint 5 -->
@@ -59,5 +55,4 @@
       </command_interface>
       <state_interface name="position"/>
-      <state_interface name="velocity"/>
     </joint>
     <!-- Joint 6 -->
@@ -68,5 +63,4 @@
       </command_interface>
       <state_interface name="position"/>
-      <state_interface name="velocity"/>
     </joint>
     <!-- Joint 7 -->
@@ -77,5 +71,4 @@
       </command_interface>
       <state_interface name="position"/>
-      <state_interface name="velocity"/>
     </joint>
     <!-- Gripper Finger Joint 1 -->
@@ -86,5 +79,4 @@
       </command_interface>
       <state_interface name="position"/>
-      <state_interface name="velocity"/>
     </joint>
     <!-- Gripper Finger Joint 2 (Mimics Joint 1) -->

File: panda_description/urdf/sensors.xacro (robot description, xacro)
@@ -12,5 +12,5 @@
                 <box size="0.1 0.1 0.05"/>
             </geometry>
-            <material name="matte_brown"/>
+            <material name="red"/>
         </visual>
         <collision>
@@ -19,5 +19,5 @@
                 <box size="0.1 0.1 0.05"/>
             </geometry>
-            <material name="matte_brown"/>
+            <material name="red"/>
         </collision>
     </link>
@@ -33,3 +33,26 @@
         <origin xyz="0 0 0" rpy="${-pi/2} 0 ${-pi/2}"/>
     </joint>
+    <gazebo reference="camera_link">
+        <sensor name="camera" type="camera">
+            <pose>0 0 0 0 1.57 0</pose>
+            <visualize>true</visualize>
+            <update_rate>10.0</update_rate>
+            <alwaysOn>true</alwaysOn>
+            <topic>camera/image_raw</topic>
+            <gz_frame_id>camera_link_optical</gz_frame_id>
+            <camera name="intel_realsense_r200">
+                <camera_info_topic>camera/camera_info</camera_info_topic>
+                <horizontal_fov>1.3962634</horizontal_fov>
+                <image>
+                    <width>640</width>
+                    <height>480</height>
+                    <format>R8G8B8</format>
+                </image>
+                <clip>
+                    <near>0.05</near>
+                    <far>8.0</far>
+                </clip>
+            </camera>
+        </sensor>
+  </gazebo>
 </robot>

Commit message: Overlay my recent local changes

File: panda_description/urdf/arm.xacro (robot description, xacro)
@@ -294,7 +294,7 @@
     <child link="panda_rightfinger"/>
     <origin rpy="0 0 0" xyz="0 0 0.0584"/>
-    <axis xyz="0 1 0"/>
+    <axis xyz="0 -1 0"/>
     <limit effort="30.0" lower="0.0" upper="0.04" velocity="10.0"/>
-    <mimic joint="panda_finger_joint1" multiplier="-1"/>
+    <!-- <mimic joint="panda_finger_joint1" multiplier="-1"/> -->
   </joint>
 </robot>

File: panda_description/urdf/panda.urdf.xacro (robot description, xacro)
@@ -2,5 +2,5 @@
 <robot name="panda" xmlns:xacro="http://www.ros.org/wiki/xacro">
   <xacro:include filename="$(find panda_description)/urdf/arm.xacro" />
-  <!-- <xacro:include filename="$(find panda_description)/urdf/sensors.xacro" /> -->
+  <xacro:include filename="$(find panda_description)/urdf/sensors.xacro" />
   <xacro:include filename="$(find panda_description)/urdf/gazebo.xacro" />
   <xacro:include filename="$(find panda_description)/urdf/ros2control.xacro" />

File: panda_description/urdf/ros2control.xacro (robot description, xacro)
@@ -82,6 +82,9 @@
     <!-- Gripper Finger Joint 2 (Mimics Joint 1) -->
     <joint name="panda_finger_joint2">
-      <param name="mimic">panda_finger_joint1</param>
-      <param name="multiplier">-1</param>
+      <command_interface name="position">
+        <param name="min">0.0</param>
+        <param name="max">0.04</param>
+      </command_interface>
+      <state_interface name="position"/>
     </joint>
   </ros2_control>
