Commit message: vision added

File: panda_description/urdf/arm.xacro (robot description, xacro)
@@ -1,7 +1,4 @@
 <?xml version="1.0" ?>
 <robot name="panda" xmlns:xacro="http://www.ros.org/wiki/xacro">
-  <material name="red">
-    <color rgba="1.0 0.0 0.0 1.000"/>
-  </material>
   <!-- World Frame -->
   <link name="world"/>

File: panda_description/urdf/panda.urdf.xacro (robot description, xacro)
@@ -1,4 +1,5 @@
 <?xml version="1.0"?>
 <robot name="panda" xmlns:xacro="http://www.ros.org/wiki/xacro">
+  <xacro:include filename="$(find panda_description)/urdf/materials.xacro" />
   <xacro:include filename="$(find panda_description)/urdf/arm.xacro" />
   <xacro:include filename="$(find panda_description)/urdf/sensors.xacro" />

File: panda_description/urdf/sensors.xacro (robot description, xacro)
@@ -23,5 +23,5 @@
     </link>
     <joint name="camera_joint" type="fixed">
-        <origin xyz="0.5 0 1.5" rpy="0.0 0.0 0.0"/>
+        <origin xyz="0.6 0 1.0" rpy="0.0 0.0 0.0"/>
         <parent link="panda_link0"/>
         <child link="camera_link"/>
@@ -43,8 +43,8 @@
             <camera name="intel_realsense_r200">
                 <camera_info_topic>camera/camera_info</camera_info_topic>
-                <horizontal_fov>1.3962634</horizontal_fov>
+                <horizontal_fov>1.0</horizontal_fov>
                 <image>
                     <width>640</width>
-                    <height>480</height>
+                    <height>320</height>
                     <format>R8G8B8</format>
                 </image>
